File: ExpansionBay ExtensionCard Module/Framework-ExpansionBay-IO-Module/Framework-ExpansionBay-IO-Module.kicad_pcb (KiCad board)
At the start: 2 copper layers, 118.7 x 72.5 mm, 20 parts, among them U1 UPD720201K8-701-BAC-A, U2 CYPD4126-40LQXIT, X1 Framework-FX-Beam, X2 Fan0, X3 Fan1, X4 USB_A, X5 USB_C_Receptacle, X6 USB_C_Receptacle, X7 USB_C_Receptacle, X8 USB_C_Receptacle

Commit message: partial redesign
Parts:
- removed the REF** at (211.4, 53.9)
- removed the REF** at (103.8, 53.9)
- added C1: 100n, Capacitor_SMD:C_0805_2012Metric, F.Cu at (163.8, 106.5)
- added C2: 100n, Capacitor_SMD:C_0805_2012Metric, F.Cu at (165.8, 106.5)
- added C3: 100n, Capacitor_SMD:C_0805_2012Metric, F.Cu at (167.8, 106.5)
- added C4: 100n, Capacitor_SMD:C_0805_2012Metric, F.Cu at (169.8, 106.5)
- added C5: 1u, Capacitor_SMD:C_0805_2012Metric, F.Cu at (189.7, 105.5)
- added C51: 100n, Capacitor_SMD:C_0805_2012Metric, F.Cu at (184.6, 95.5)
- added C52: 100n, Capacitor_SMD:C_0805_2012Metric, F.Cu at (184.6, 93.5)
- added C53: 100n, Capacitor_SMD:C_0805_2012Metric, F.Cu at (189.7, 95.7)
- added C54: 100n, Capacitor_SMD:C_0805_2012Metric, F.Cu at (189.7, 97.7)
- added C6: 1u, Capacitor_SMD:C_0805_2012Metric, F.Cu at (189.7, 99.7)
- added C61: 100n, Capacitor_SMD:C_0805_2012Metric, F.Cu at (152.4, 95.5)
- added C62: 100n, Capacitor_SMD:C_0805_2012Metric, F.Cu at (152.4, 93.5)
- added C63: 100n, Capacitor_SMD:C_0805_2012Metric, F.Cu at (152.4, 97.5)
- added C64: 100n, Capacitor_SMD:C_0805_2012Metric, F.Cu at (152.4, 99.5)
- added C71: 100n, Capacitor_SMD:C_0805_2012Metric, F.Cu at (122.5, 95.4)
- added C72: 100n, Capacitor_SMD:C_0805_2012Metric, F.Cu at (122.5, 93.5)
- added C73: 100n, Capacitor_SMD:C_0805_2012Metric, F.Cu at (127.7, 95.7)
- added C74: 100n, Capacitor_SMD:C_0805_2012Metric, F.Cu at (127.7, 97.7)
- added C81: 100n, Capacitor_SMD:C_0805_2012Metric, F.Cu at (141.6, 101.2)
- added C82: 100n, Capacitor_SMD:C_0805_2012Metric, F.Cu at (141.6, 103.1)
- added C83: 100n, Capacitor_SMD:C_0805_2012Metric, F.Cu at (142.3, 96.5)
- added C84: 100n, Capacitor_SMD:C_0805_2012Metric, F.Cu at (144.3, 96.5)
- added R1: 1k60, Resistor_SMD:R_0805_2012Metric, F.Cu at (176.9, 94.3)
- added R10: 10k, Resistor_SMD:R_0805_2012Metric, F.Cu at (159.8, 106.5)
- added R11: 10k, Resistor_SMD:R_0805_2012Metric, F.Cu at (161.8, 106.5)
- added R12: 10k, Resistor_SMD:R_0805_2012Metric, F.Cu at (182.6, 105.6)
- added R13: 10k, Resistor_SMD:R_0805_2012Metric, F.Cu at (186.0, 105.6)
- added R14: 10k, Resistor_SMD:R_0805_2012Metric, F.Cu at (189.7, 103.5)
- added R15: 15k-16k, Resistor_SMD:R_0805_2012Metric, F.Cu at (189.7, 101.6)
- added R16: 10k, Resistor_SMD:R_0805_2012Metric, F.Cu at (101.6, 71.8)
- added R17: 10k, Resistor_SMD:R_0805_2012Metric, F.Cu at (101.6, 76.0)
- added R2: 10k, Resistor_SMD:R_0805_2012Metric, F.Cu at (177.0, 96.3)
- added R3: 10k, Resistor_SMD:R_0805_2012Metric, F.Cu at (177.0, 98.2)
- added R4: 10k, Resistor_SMD:R_0805_2012Metric, F.Cu at (177.0, 100.2)
- added R5: 47k, Resistor_SMD:R_0805_2012Metric, F.Cu at (177.0, 102.1)
- added R6: 10k, Resistor_SMD:R_0805_2012Metric, F.Cu at (177.0, 104.0)
- added R62: 100k, Resistor_SMD:R_0805_2012Metric, F.Cu at (179.8, 82.8)
- added R63: 100k, Resistor_SMD:R_0805_2012Metric, F.Cu at (177.9, 86.2)
- added R64: 100k, Resistor_SMD:R_0805_2012Metric, F.Cu at (181.7, 86.2)
- added R65: 100k, Resistor_SMD:R_0805_2012Metric, F.Cu at (179.8, 86.2)
- added R66: 100k, Resistor_SMD:R_0805_2012Metric, F.Cu at (181.7, 82.8)
- added R67: 100k, Resistor_SMD:R_0805_2012Metric, F.Cu at (177.9, 82.8)
- added R7: 330k, Resistor_SMD:R_0805_2012Metric, F.Cu at (177.0, 105.9)
- added R72: 100k, Resistor_SMD:R_0805_2012Metric, F.Cu at (147.8, 82.9)
- added R73: 100k, Resistor_SMD:R_0805_2012Metric, F.Cu at (146.8, 86.3)
- added R74: 100k, Resistor_SMD:R_0805_2012Metric, F.Cu at (150.6, 86.3)
- added R75: 100k, Resistor_SMD:R_0805_2012Metric, F.Cu at (148.7, 86.3)
- added R76: 100k, Resistor_SMD:R_0805_2012Metric, F.Cu at (149.7, 82.9)
- added R8: 100k, Resistor_SMD:R_0805_2012Metric, F.Cu at (156.0, 106.5)
- added R82: 100k, Resistor_SMD:R_0805_2012Metric, F.Cu at (116.8, 82.8)
- added R83: 100k, Resistor_SMD:R_0805_2012Metric, F.Cu at (115.8, 86.2)
- added R84: 100k, Resistor_SMD:R_0805_2012Metric, F.Cu at (119.7, 86.2)
- added R85: 100k, Resistor_SMD:R_0805_2012Metric, F.Cu at (117.8, 86.2)
- added R86: 100k, Resistor_SMD:R_0805_2012Metric, F.Cu at (118.7, 82.8)
- added REF**: ExpansionCard-Rail&Lock, Framework-ExpansionBay-IOModule:ExpansionCard-Rail&Lock, F.Cu at (203.2, 83.0)
- added REF**: ExpansionCard-Rail&Lock, Framework-ExpansionBay-IOModule:ExpansionCard-Rail&Lock, F.Cu at (141.2, 83.0)
- added REF**: ExpansionCard-Rail&Lock, Framework-ExpansionBay-IOModule:ExpansionCard-Rail&Lock, F.Cu at (110.3, 83.0)
- added REF**: ExpansionCard-Rail&Lock, Framework-ExpansionBay-IOModule:ExpansionCard-Rail&Lock, F.Cu at (172.2, 83.0)
- added U3: MCP1727-ADJxMF, Package_DFN_QFN:DFN-8-1EP_3x3mm_P0.65mm_EP1.55x2.4mm, F.Cu at (184.2, 102.7)
- added U51: XC8107, Package_TO_SOT_SMD:SOT-23-5, F.Cu at (189.7, 93.0)
- added U52: FUSB303BTMX, Package_DFN_QFN:Texas_X2QFN-12_1.6x1.6mm_P0.4mm, B.Cu at (183.0, 92.9)
- added U53: FUSB340TMX, Framework-ExpansionBay-IOModule:QFN40P200X280X40-19N, B.Cu at (187.6, 92.5)
- added U61: XC8107, Package_TO_SOT_SMD:SOT-23-5, F.Cu at (158.3, 93.0)
- added U62: FUSB303BTMX, Package_DFN_QFN:Texas_X2QFN-12_1.6x1.6mm_P0.4mm, B.Cu at (152.0, 93.0)
- added U63: FUSB340TMX, Framework-ExpansionBay-IOModule:QFN40P200X280X40-19N, B.Cu at (156.6, 92.5)
- added U71: XC8107, Package_TO_SOT_SMD:SOT-23-5, F.Cu at (127.7, 93.0)
- added U72: FUSB303BTMX, Package_DFN_QFN:Texas_X2QFN-12_1.6x1.6mm_P0.4mm, B.Cu at (121.0, 92.9)
- added U73: FUSB340TMX, Framework-ExpansionBay-IOModule:QFN40P200X280X40-19N, B.Cu at (125.6, 92.5)
- added U81: XC8107, Package_TO_SOT_SMD:SOT-23-5, F.Cu at (139.7, 96.6)
- added X10: FOXCONN 3VM11201-D730-7H, Framework-ExpansionBay-IOModule:Mini DP FOXCONN 3VM11201-D730-7H, F.Cu at (109.3, 54.3)
- added X9: Molex-SFF8612-OcuLink-1719821142, Framework-ExpansionBay-IOModule:MOLEX_1719821142, F.Cu at (211.1, 55.7)
- added Y1: 24MHz, Crystal:Crystal_SMD_EuroQuartz_MT-4Pin_3.2x2.5mm, B.Cu at (176.6, 96.4)
- U2: value CYPD4126-40LQXIT -> 24LC32A-I/SN; footprint Package_DFN_QFN:QFN-40-1EP_6x6mm_P0.5mm_EP4.6x4.6mm -> Package_SO:SOIC-8_3.9x4.9mm_P1.27mm
- X8: value USB_C_Receptacle -> Expansion-USB3; footprint Framework-ExpansionBay-IOModule:Amphenol-USBC-10137062-00021LF -> Framework-ExpansionBay-IOModule:DS1015-02-12R6
- moved U2 106.8 mm to (143.5, 107.4)
- moved X8 87.9 mm to (133.4, 102.6), turned to 0 degrees
- moved U1 68.9 mm to (166.4, 98.0), turned to 90 degrees
- moved R9 14.4 mm to (157.9, 106.5), turned to 90 degrees
- moved X4 9.54 mm to (117.5, 103.0)
- moved REF** 2.15 mm to (187.7, 62.0)
- moved REF** 2.15 mm to (156.7, 62.0)
- moved X5 2.15 mm to (187.7, 87.2)
- moved X6 2.15 mm to (156.7, 87.2)
- moved REF** 2.15 mm to (125.7, 62.0)
- moved X7 1.95 mm to (125.7, 87.2)
- renumbered R1 to R9
Connections:
- net /Power Connect/GPIO0_EC renamed GPIO0_EC
- net /Power Connect/GPIO1_EC renamed GPIO1_EC
- net Net-(X5-VBUS-PadA4) renamed USB1_VBUS
- net Net-(X6-VBUS-PadA4) renamed USB2_VBUS
- net Net-(X7-VBUS-PadA4) renamed USB3_VBUS
- U1 pad 20: unconnected-(U1-OCI4B-Pad20) -> Net-(U1-OCI4B)
- U1 pad 21: unconnected-(U1-PPON4-Pad21) -> Net-(U1-PPON4)
- U1 pad 22: unconnected-(U1-OCI3B-Pad22) -> Net-(U1-OCI3B)
- U1 pad 23: unconnected-(U1-PPON3-Pad23) -> Net-(U1-PPON3)
- U1 pad 24: unconnected-(U1-OCI2B-Pad24) -> Net-(U1-OCI2B)
- U1 pad 25: unconnected-(U1-PPON2-Pad25) -> Net-(U1-PPON2)
- U1 pad 26: unconnected-(U1-OCI1B-Pad26) -> Net-(U1-OCI1B)
- U1 pad 27: unconnected-(U1-PPON1-Pad27) -> Net-(U1-PPON1)
- U1 pad 3: unconnected-(U1-PEWAKEB-Pad3) -> Net-(U1-PEWAKEB)
- U1 pad 7: PEX_RX0+ -> Net-(U1-PETXP)
- U1 pad 8: PEX_RX0- -> Net-(U1-PETXN)
- U2 pad 1: unconnected-(U2-SWD_IO/AR_RST#-Pad1) -> GND
- U2 pad 2: unconnected-(U2-SWD_CLK/I2C_CFG_EC-Pad2) -> GND
- U2 pad 3: unconnected-(U2-I2C_SDA_SCB1_AR-Pad3) -> GND
- U2 pad 4: unconnected-(U2-I2C_SCL_SCB1_AR-Pad4) -> GND
- U2 pad 5: unconnected-(U2-I2C_INT_AR_P0-Pad5) -> I2C_SDA_EC
- U2 pad 6: unconnected-(U2-P1.5-Pad6) -> I2C_SCL_EC
- U2 pad 7: unconnected-(U2-CC2_P0-Pad7) -> Net-(U2-WP)
- U2 pad 8: unconnected-(U2-V5V_P0-Pad8) -> +3V3
- X1 pad D-1: unconnected-(X1B-PEX_RX1N-PadD-1) -> PEX_RX1-
- X1 pad D-10: unconnected-(X1B-PEX_TX1N-PadD-10) -> PEX_TX1-
- X1 pad D-11: unconnected-(X1B-PEX_TX1P-PadD-11) -> PEX_TX1+
- X1 pad D-12: unconnected-(X1B-DP_A_HPD-PadD-12) -> DP_HPD
- X1 pad D-14: unconnected-(X1B-DP_A_L1#-PadD-14) -> DP_L1-
- X1 pad D-15: unconnected-(X1B-DP_A_L1-PadD-15) -> DP_L1+
- X1 pad D-17: unconnected-(X1B-DP_A_L0#-PadD-17) -> DP_L0-
- X1 pad D-18: unconnected-(X1B-DP_A_L0-PadD-18) -> DP_L0+
- X1 pad D-2: unconnected-(X1B-PEX_RX1P-PadD-2) -> PEX_RX1+
- X1 pad D-20: unconnected-(X1B-DP_A_AUX#-PadD-20) -> DP_AUX-
- X1 pad D-21: unconnected-(X1B-DP_A_AUX-PadD-21) -> DP_AUX+
- X1 pad D-22: unconnected-(X1B-GPIO3_EC-PadD-22) -> EC_GPIO3
- X1 pad D-23: unconnected-(X1B-PEX_RX3N-PadD-23) -> PEX_RX3-
- X1 pad D-24: unconnected-(X1B-PEX_RX3P-PadD-24) -> PEX_RX3+
- X1 pad D-26: unconnected-(X1B-PEX_RX2N-PadD-26) -> PEX_RX2-
- X1 pad D-27: unconnected-(X1B-PEX_RX2P-PadD-27) -> PEX_RX2+
- X1 pad D-29: unconnected-(X1B-PEX_TX2P-PadD-29) -> PEX_TX2+
- X1 pad D-30: unconnected-(X1B-PEX_TX2N-PadD-30) -> PEX_TX2-
- X1 pad D-32: unconnected-(X1B-PEX_TX3N-PadD-32) -> PEX_TX3-
- X1 pad D-33: unconnected-(X1B-PEX_TX3P-PadD-33) -> PEX_TX3+
- X1 pad D-35: unconnected-(X1B-TH_ALERT#-PadD-35) -> EC_TH_ALERT
- X1 pad D-36: unconnected-(X1B-PNL_PWR_EN-PadD-36) -> PNL_PWR_EN
- X1 pad D-37: unconnected-(X1B-TH_OVERT#-PadD-37) -> EC_TH_OVERTEMP
- X1 pad D-39: unconnected-(X1B-DGPU_PWM_SEL-PadD-39) -> DGPU_PWM_SEL
- X1 pad D-40: unconnected-(X1B-PNL_BL_PWM-PadD-40) -> PNL_BL_PWM
- X1 pad D-41: unconnected-(X1B-PNL_BL_EN-PadD-41) -> PNL_BL_EN
- X1 pad D-42: unconnected-(X1B-PEX_RX4P-PadD-42) -> PEX_RX4+
- X1 pad D-43: unconnected-(X1B-PEX_RX4N-PadD-43) -> PEX_RX4-
- X1 pad D-45: unconnected-(X1B-PEX_RX5P-PadD-45) -> PEX_RX5+
- X1 pad D-46: unconnected-(X1B-PEX_RX5N-PadD-46) -> PEX_RX5-
- X1 pad D-48: unconnected-(X1B-PEX_TX5N-PadD-48) -> PEX_TX5-
- X1 pad D-49: unconnected-(X1B-PEX_TX5P-PadD-49) -> PEX_TX5+
- X1 pad D-51: unconnected-(X1B-PEX_TX4P-PadD-51) -> PEX_TX4+
- X1 pad D-52: unconnected-(X1B-PEX_TX4N-PadD-52) -> PEX_TX4-
- X1 pad D-53: unconnected-(X1B-GPIO2_EC-PadD-53) -> EC_GPIO2
- X1 pad D-58: unconnected-(X1B-DP_A_L3#-PadD-58) -> DP_L3-
- X1 pad D-59: unconnected-(X1B-DP_A_L3-PadD-59) -> DP_L3+
- X1 pad D-61: unconnected-(X1B-DP_A_L2#-PadD-61) -> DP_L2-
- X1 pad D-62: unconnected-(X1B-DP_A_L2-PadD-62) -> DP_L2+
- X1 pad D-63: unconnected-(X1B-ID1-PadD-63) -> Net-(X1B-ID1)
- X1 pad D-64: unconnected-(X1B-PEX_RX6P-PadD-64) -> PEX_RX6+
- X1 pad D-65: unconnected-(X1B-PEX_RX6N-PadD-65) -> PEX_RX6-
- X1 pad D-67: unconnected-(X1B-PEX_RX7N-PadD-67) -> PEX_RX7-
- X1 pad D-68: unconnected-(X1B-PEX_RX7P-PadD-68) -> PEX_RX7+
- X1 pad D-7: PEX_TX0- -> Net-(X1B-PEX_TX0N)
- X1 pad D-70: unconnected-(X1B-PEX_TX7N-PadD-70) -> PEX_TX7-
- X1 pad D-71: unconnected-(X1B-PEX_TX7P-PadD-71) -> PEX_TX7+
- X1 pad D-73: unconnected-(X1B-PEX_TX6P-PadD-73) -> PEX_TX6+
- X1 pad D-74: unconnected-(X1B-PEX_TX6N-PadD-74) -> PEX_TX6-
- X1 pad D-8: PEX_TX0+ -> Net-(X1B-PEX_TX0P)
- X1 pad P-44: unconnected-(X1A-I2C_CLK_ALW-PadP-44) -> I2C_SCL_EC
- X1 pad P-45: unconnected-(X1A-I2C_SDA_ALW-PadP-45) -> I2C_SDA_EC
- X1 pad P-47: unconnected-(X1A-EXT_SSD1_RST#-PadP-47) -> EXT_SSD1_RST
- X1 pad P-48: unconnected-(X1A-EXT_SSD2_RST#-PadP-48) -> EXT_SSD2_RST
- X1 pad P-58: unconnected-(X1A-I2C_INT_ALW-PadP-58) -> I2C_INT_EC
- X1 pad P-59: unconnected-(X1A-EXT_SSD2_CLK_REQ#-PadP-59) -> EXT_SSD2_CLK_REQ
- X1 pad P-62: unconnected-(X1A-PWR_EN-PadP-62) -> PWR_EN
- X1 pad P-63: unconnected-(X1A-DDS_CLK-PadP-63) -> DDS_CLK
- X1 pad P-73: unconnected-(X1A-DDS_SDA-PadP-73) -> DDS_SDA
- X1 pad P-74: unconnected-(X1A-PWR_GOOD-PadP-74) -> PWR_GOOD
- X5 pad A10: USB1_RX- -> USB1_SSRX2-
- X5 pad A11: USB1_RX+ -> USB1_SSRX2+
- X5 pad A2: USB1_TX+ -> USB1_SSTX1+
- X5 pad A3: USB1_TX- -> USB1_SSTX1-
- X5 pad A5: unconnected-(X5-CC1-PadA5) -> USB1_CC1
- X5 pad B10: USB1_RX- -> USB1_SSRX1-
- X5 pad B11: USB1_RX+ -> USB1_SSRX1+
- X5 pad B2: USB1_TX+ -> USB1_SSTX2+
- X5 pad B3: USB1_TX- -> USB1_SSTX2-
- X5 pad B5: unconnected-(X5-CC2-PadB5) -> USB1_CC2
- X6 pad A10: USB2_RX- -> USB2_SSRX2-
- X6 pad A11: USB2_RX+ -> USB2_SSRX2+
- X6 pad A2: USB2_TX+ -> USB2_SSTX1+
- X6 pad A3: USB2_TX- -> USB2_SSTX1-
- X6 pad A5: unconnected-(X6-CC1-PadA5) -> USB2_CC1
- X6 pad B10: USB2_RX- -> USB2_SSRX1-
- X6 pad B11: USB2_RX+ -> USB2_SSRX1+
- X6 pad B2: USB2_TX+ -> USB2_SSTX2+
- X6 pad B3: USB2_TX- -> USB2_SSTX2-
- X6 pad B5: unconnected-(X6-CC2-PadB5) -> USB2_CC2
- X7 pad A10: USB3_RX- -> USB3_SSRX2-
- X7 pad A11: USB3_RX+ -> USB3_SSRX2+
- X7 pad A2: USB3_TX+ -> USB3_SSTX1+
- X7 pad A3: USB3_TX- -> USB3_SSTX1-
- X7 pad A5: unconnected-(X7-CC1-PadA5) -> USB3_CC1
- X7 pad B10: USB3_RX- -> USB3_SSRX1-
- X7 pad B11: USB3_RX+ -> USB3_SSRX1+
- X7 pad B2: USB3_TX+ -> USB3_SSTX2+
- X7 pad B3: USB3_TX- -> USB3_SSTX2-
- X7 pad B5: unconnected-(X7-CC2-PadB5) -> USB3_CC2
Routing:
- net GND: track 0.00 -> 684.8 mm, vias 0 -> 161
- net +5V: track 0.00 -> 232.6 mm, vias 0 -> 20
- net DP_AUX-: track 0.00 -> 133.2 mm, vias 0 -> 3
- net DP_AUX+: track 0.00 -> 133.2 mm, vias 0 -> 3
- net DP_L2+: track 0.00 -> 125.9 mm, vias 0 -> 2
- net DP_L2-: track 0.00 -> 125.9 mm, vias 0 -> 2
- net DP_L0-: track 0.00 -> 124.7 mm, vias 0 -> 1
- net DP_L0+: track 0.00 -> 122.8 mm, vias 0 -> 3
- net DP_L3+: track 0.00 -> 122.6 mm, vias 0 -> 2
- net DP_L3-: track 0.00 -> 122.6 mm, vias 0 -> 2
- net DP_L1+: track 0.00 -> 118.4 mm, vias 0 -> 2
- net DP_L1-: track 0.00 -> 118.4 mm, vias 0 -> 2
- net DP_HPD: track 0.00 -> 117.8 mm, vias 0 -> 2
- net PEX_TX5-: track 0.00 -> 112.6 mm, vias 0 -> 2
- net PEX_TX5+: track 0.00 -> 108.0 mm, vias 0 -> 2
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- added copper zone on In1.Cu, net +3V3
- added copper zone on B.Cu, net GND
- added copper zone on In1.Cu, net GND
- added copper zone on In2.Cu, net GND
Other:
- copper layers 2 -> 4
