File: ExpansionBay ExtensionCard Module/Framework-ExpansionBay-IO-Module/dataConnector.kicad_sch (KiCad schematic)
At the start: 6 parts, among them X1 Framework-FX-Beam, X5 USB_C_Receptacle, X6 USB_C_Receptacle, X7 USB_C_Receptacle

Commit message: partial redesign
Parts:
- added R7: 330k, Resistor_SMD:R_0805_2012Metric, symbol Device:R
- C3: renamed from C18; footprint (none) -> Capacitor_SMD:C_0805_2012Metric
- C4: renamed from C17; footprint (none) -> Capacitor_SMD:C_0805_2012Metric
Connections:
- net GND: now also R7.2
- net PEX_RX1-: now reaches X1.D-1 (PEX_RX1N)
- net PEX_TX1-: now reaches X1.D-10 (PEX_TX1N)
- net PEX_TX1+: now reaches X1.D-11 (PEX_TX1P)
- net PEX_RX1+: now reaches X1.D-2 (PEX_RX1P)
- net EC_GPIO3: now reaches X1.D-22 (GPIO3_EC)
- net PEX_RX3-: now reaches X1.D-23 (PEX_RX3N)
- net PEX_RX3+: now reaches X1.D-24 (PEX_RX3P)
- net PEX_RX2-: now reaches X1.D-26 (PEX_RX2N)
- net PEX_RX2+: now reaches X1.D-27 (PEX_RX2P)
- net PEX_TX2+: now reaches X1.D-29 (PEX_TX2P)
- net PEX_TX2-: now reaches X1.D-30 (PEX_TX2N)
- net PEX_TX3-: now reaches X1.D-32 (PEX_TX3N)
- net PEX_TX3+: now reaches X1.D-33 (PEX_TX3P)
- net EC_TH_ALERT: now reaches X1.D-35 (TH_ALERT#)
- net PNL_PWR_EN: now reaches X1.D-36 (PNL_PWR_EN)
- net EC_TH_OVERTEMP: now reaches X1.D-37 (TH_OVERT#)
- net DGPU_PWM_SEL: now reaches X1.D-39 (DGPU_PWM_SEL)
- net PNL_BL_PWM: now reaches X1.D-40 (PNL_BL_PWM)
- net PNL_BL_EN: now reaches X1.D-41 (PNL_BL_EN)
- net PEX_RX4+: now reaches X1.D-42 (PEX_RX4P)
- net PEX_RX4-: now reaches X1.D-43 (PEX_RX4N)
- net PEX_RX5+: now reaches X1.D-45 (PEX_RX5P)
- net PEX_RX5-: now reaches X1.D-46 (PEX_RX5N)
- net PEX_TX5-: now reaches X1.D-48 (PEX_TX5N)
- net PEX_TX5+: now reaches X1.D-49 (PEX_TX5P)
- net PEX_TX4+: now reaches X1.D-51 (PEX_TX4P)
- net PEX_TX4-: now reaches X1.D-52 (PEX_TX4N)
- net EC_GPIO2: now reaches X1.D-53 (GPIO2_EC)
- net at X1.D-63 (ID1): now also R7.1
- net PEX_RX6+: now reaches X1.D-64 (PEX_RX6P)
- net PEX_RX6-: now reaches X1.D-65 (PEX_RX6N)
- net PEX_RX7-: now reaches X1.D-67 (PEX_RX7N)
- net PEX_RX7+: now reaches X1.D-68 (PEX_RX7P)
- net PEX_TX7-: now reaches X1.D-70 (PEX_TX7N)
- net PEX_TX7+: now reaches X1.D-71 (PEX_TX7P)
- net PEX_TX6+: now reaches X1.D-73 (PEX_TX6P)
- net PEX_TX6-: now reaches X1.D-74 (PEX_TX6N)
- net USB2_CC1: now reaches X6.A5 (CC1)
- net USB2_CC2: now reaches X6.B5 (CC2)
- net USB1_CC1: now reaches X5.A5 (CC1)
- net USB1_CC2: now reaches X5.B5 (CC2)
- net USB3_CC1: now reaches X7.A5 (CC1)
- net USB3_CC2: now reaches X7.B5 (CC2)
- net USB1_RX+ renamed USB1_SSRX1+
- net USB1_SSRX1+: no longer X5.A11 (RX2+)
- net USB1_RX- renamed USB1_SSRX1-
- net USB1_SSRX1-: no longer X5.A10 (RX2-)
- net USB1_TX+ renamed USB1_SSTX1+
- net USB1_SSTX1+: no longer X5.B2 (TX2+)
- net USB1_TX- renamed USB1_SSTX1-
- net USB1_SSTX1-: no longer X5.B3 (TX2-)
- net USB2_RX+ renamed USB2_SSRX1+
- net USB2_SSRX1+: no longer X6.A11 (RX2+)
- net USB2_RX- renamed USB2_SSRX1-
- net USB2_SSRX1-: no longer X6.A10 (RX2-)
- net USB2_TX+ renamed USB2_SSTX1+
- net USB2_SSTX1+: no longer X6.B2 (TX2+)
- net USB2_TX- renamed USB2_SSTX1-
- net USB2_SSTX1-: no longer X6.B3 (TX2-)
- net USB3_RX+ renamed USB3_SSRX1+
- net USB3_SSRX1+: no longer X7.A11 (RX2+)
- net USB3_RX- renamed USB3_SSRX1-
- net USB3_SSRX1-: no longer X7.A10 (RX2-)
- net USB3_TX+ renamed USB3_SSTX1+
- net USB3_SSTX1+: no longer X7.B2 (TX2+)
- net USB3_TX- renamed USB3_SSTX1-
- net USB3_SSTX1-: no longer X7.B3 (TX2-)
- new net USB1_SSRX2+: X5.A11 (RX2+)
- new net USB1_SSRX2-: X5.A10 (RX2-)
- new net USB1_SSTX2+: X5.B2 (TX2+)
- new net USB1_SSTX2-: X5.B3 (TX2-)
- new net USB2_SSRX2+: X6.A11 (RX2+)
- new net USB2_SSRX2-: X6.A10 (RX2-)
- new net USB2_SSTX2+: X6.B2 (TX2+)
- new net USB2_SSTX2-: X6.B3 (TX2-)
- new net USB3_SSRX2+: X7.A11 (RX2+)
- new net USB3_SSRX2-: X7.A10 (RX2-)
- new net USB3_SSTX2+: X7.B2 (TX2+)
- new net USB3_SSTX2-: X7.B3 (TX2-)
