File: ExpansionBay ExtensionCard Module/Framework-ExpansionBay-IO-Module/powerConnect.kicad_sch (KiCad schematic)
At the start: 7 parts, among them X1 Framework-FX-Beam, X2 Fan0, X3 Fan1, X4 USB_A, X8 USB_C_Receptacle

Commit message: partial redesign
Parts:
- removed C1: 1u, symbol Device:C
- removed X2: Fan0, Framework-ExpansionBay:Molex-52746-0471, symbol Connector_Generic:Conn_01x04
- removed X3: Fan1, Framework-ExpansionBay:Molex-52746-0471, symbol Connector_Generic:Conn_01x04
- removed X4: USB_A, Framework-ExpansionBay-IOModule:Würth-USB2-629104190121, symbol Connector:USB_A
- removed X8: USB_C_Receptacle, Framework-ExpansionBay-IOModule:Amphenol-USBC-10137062-00021LF, symbol Framework-ExpansionBay-IOModule:USB_C_Receptacle
- added C5, C6: 1u, Capacitor_SMD:C_0805_2012Metric, symbol Device:C
- added R12, R13, R14, R16, R17: 10k, Resistor_SMD:R_0805_2012Metric, symbol Device:R
- added R15: 15k-16k, Resistor_SMD:R_0805_2012Metric, symbol Device:R
- added U3: MCP1727-ADJxMF, Package_DFN_QFN:DFN-8-1EP_3x3mm_P0.65mm_EP1.55x2.4mm, symbol Regulator_Linear:MCP1727-ADJxMF
- added X10: FOXCONN 3VM11201-D730-7H, Framework-ExpansionBay-IOModule:Mini DP FOXCONN 3VM11201-D730-7H, symbol Framework-ExpansionBay-IOModule:Mini_Displayport
- added X9: Molex-SFF8612-OcuLink-1719821142, Framework-ExpansionBay-IOModule:MOLEX_1719821142, symbol Framework-ExpansionBay-IOModule:Molex-SFF8612-OcuLink-1719821142
- renumbered R1 to R9
Connections:
- net +3V3: now also R12.2, R13.2, U3.1 (Vin), U3.2 (Vin), X10.20 (DP_PWR), X9.A1 (3V3), X9.B21 (3V3)
- net +5V: now also X9.A21 (5V), X9.B1 (5V)
- net GND: now also C5.1, C6.1, R14.1, R16.2, R17.2, U3.4 (GND), U3.9 (GND), X10.1 (GND), X10.13 (GND), X10.14 (GND), X10.19 (GND), X10.7 (GND), X10.8 (GND), X10.G (GND), X9.A11 (GND), X9.A14 (GND), X9.A17 (GND), X9.A2 (GND), X9.A20 (GND), X9.A5 (GND), X9.A8 (GND), X9.B11 (GND), X9.B14 (GND), X9.B17 (GND), X9.B2 (GND), X9.B20 (GND), X9.B5 (GND), X9.B8 (GND), X9.S1 (SHIELD), X9.S2 (SHIELD), X9.S3 (SHIELD), X9.S4 (SHIELD)
- net EXT_SSD1_RST: now reaches X1.P-47 (EXT_SSD1_RST#)
- net EXT_SSD2_RST: now reaches X1.P-48 (EXT_SSD2_RST#)
- net EXT_SSD2_CLK_REQ: now reaches X1.P-59 (EXT_SSD2_CLK_REQ#)
- net PWR_EN: now reaches X1.P-62 (PWR_EN)
- net DDS_CLK: now reaches X1.P-63 (DDS_CLK)
- net DDS_SDA: now reaches X1.P-73 (DDS_SDA)
- net PWR_GOOD: now reaches X1.P-74 (PWR_GOOD)
- new net: R16.1, X10.6 (CONFIG2)
- new net: C5.2, U3.6 (Cdelay)
- new net: R14.2, R15.1, U3.7 (ADJ)
- new net: R13.1, U3.5 (PWRGD)
- new net: R17.1, X10.4 (CONFIG1)
- new net: R12.1, U3.3 (~{SHDN})
- new net +1V0: C6.2, R15.2, U3.8 (Vout)
- new net DP_AUX+: X10.16 (AUXp)
- new net DP_AUX-: X10.18 (AUXn)
- new net DP_HPD: X10.2 (HPD)
- new net DP_L0+: X10.12 (L3n(SRC)/L0p(SNK))
- new net DP_L0-: X10.10 (L3p(SRC)/L0n(SNK))
- new net DP_L1+: X10.17 (L2n(SRC)/L1p(SNK))
- new net DP_L1-: X10.15 (L2p(SRC)/L1n(SNK))
- new net DP_L2+: X10.11 (L1n(SRC)/L2p(SNK))
- new net DP_L2-: X10.9 (L1p(SRC)/L2n(SNK))
- new net DP_L3+: X10.5 (L0n(SRC)/L3p(SNK))
- new net DP_L3-: X10.3 (L0p(SRC)/L3n(SNK))
- new net PEX_RST: X9.B12 (PERST#)
- new net PEX_RX4+: X9.A3 (PERp0)
- new net PEX_RX4-: X9.A4 (PERn0)
- new net PEX_RX5+: X9.A6 (PERp1)
- new net PEX_RX5-: X9.A7 (PERn1)
- new net PEX_RX6+: X9.A15 (PERp2)
- new net PEX_RX6-: X9.A16 (PERn2)
- new net PEX_RX7+: X9.A18 (PERp3)
- new net PEX_RX7-: X9.A19 (PERn3)
- new net PEX_TX4+: X9.B3 (PETp0)
- new net PEX_TX4-: X9.B4 (PETn0)
- new net PEX_TX5+: X9.B6 (PETp1)
- new net PEX_TX5-: X9.B7 (PETn1)
- new net PEX_TX6+: X9.B15 (PETp2)
- new net PEX_TX6-: X9.B16 (PETn2)
- new net PEX_TX7+: X9.B18 (PETp3)
- new net PEX_TX7-: X9.B19 (PETn3)
Other:
- note added: "1.05V LDO"
- note added: "Mini DP IN"
- note added: "OcuLink Connector (external)"
- note removed: "Fan Connectors"
- note removed: "USB 2.0 Internal (for dongles)"
- note removed: "USB 3.0 PD (external)"
