File: ExpansionBay ExtensionCard Module/Framework-ExpansionBay-IO-Module/usb3.kicad_sch (KiCad schematic)
At the start: 38 parts, among them U1 UPD720201K8-701-BAC-A, U3 AP2171, U4 AP2171, U5 AP2171, Y1 24MHz

Commit message: partial redesign
Parts:
- removed Y1: 24MHz, symbol Device:Crystal
- added C31: 10u, symbol Device:C_Polarized
- added C34: 120u, symbol Device:C_Polarized
- added C83, C84: 100n, Capacitor_SMD:C_0805_2012Metric, symbol Device:C
- added R81: 10k, symbol Device:R
- added U81: XC8107, Package_TO_SOT_SMD:SOT-23-5, symbol Framework-ExpansionBay-IOModule:AP2171
- added Y1: 24MHz, Crystal:Crystal_SMD_EuroQuartz_MT-4Pin_3.2x2.5mm, symbol Device:Crystal_GND24
- C1: renamed from C15; footprint (none) -> Capacitor_SMD:C_0805_2012Metric
- C2: renamed from C16; footprint (none) -> Capacitor_SMD:C_0805_2012Metric
- C51: renamed from C2; footprint (none) -> Capacitor_SMD:C_0805_2012Metric
- C52: renamed from C3; footprint (none) -> Capacitor_SMD:C_0805_2012Metric
- C53: renamed from C25; footprint (none) -> Capacitor_SMD:C_0805_2012Metric
- C54: renamed from C21; footprint (none) -> Capacitor_SMD:C_0805_2012Metric
- C61: renamed from C4; footprint (none) -> Capacitor_SMD:C_0805_2012Metric
- C62: renamed from C5; footprint (none) -> Capacitor_SMD:C_0805_2012Metric
- C63: renamed from C26; footprint (none) -> Capacitor_SMD:C_0805_2012Metric
- C64: renamed from C20; footprint (none) -> Capacitor_SMD:C_0805_2012Metric
- C71: renamed from C6; footprint (none) -> Capacitor_SMD:C_0805_2012Metric
- C72: renamed from C7; footprint (none) -> Capacitor_SMD:C_0805_2012Metric
- C73: renamed from C27; footprint (none) -> Capacitor_SMD:C_0805_2012Metric
- C74: renamed from C19; footprint (none) -> Capacitor_SMD:C_0805_2012Metric
- C81: renamed from C8; footprint (none) -> Capacitor_SMD:C_0805_2012Metric
- C82: renamed from C9; footprint (none) -> Capacitor_SMD:C_0805_2012Metric
- R1: renamed from R2; footprint (none) -> Resistor_SMD:R_0805_2012Metric
- R10: renamed from R7; footprint (none) -> Resistor_SMD:R_0805_2012Metric
- R11, R4: footprint (none) -> Resistor_SMD:R_0805_2012Metric
- R2: renamed from R3; footprint (none) -> Resistor_SMD:R_0805_2012Metric
- R3: renamed from R5; footprint (none) -> Resistor_SMD:R_0805_2012Metric
- R5: renamed from R6; footprint (none) -> Resistor_SMD:R_0805_2012Metric
- R6: renamed from R12; footprint (none) -> Resistor_SMD:R_0805_2012Metric
- U51: renamed from U3; value AP2171 -> XC8107
- U61: renamed from U4; value AP2171 -> XC8107
- U71: renamed from U5; value AP2171 -> XC8107
- renumbered R13 to R51, R14 to R61, R15 to R71
Connections:
- net +3V3: now also R81.1
- net +5V: now also C31.1, C83.2, U81.5 (IN)
- net GND: now also C31.2, C34.2, C83.1, C84.1, U81.2 (GND), Y1.2, Y1.4
- net at U1.20 (OCI4B): now also R81.2, U81.3 (FLG)
- net at U1.21 (PPON4): now also U81.4 (EN)
- net at U1.30 (XT2): now also Y1.1
- net at U1.31 (XT1): now also Y1.3
- new net USB4_VBUS: C34.1, C84.2, U81.1 (OUT)
Other:
- note removed: "USB4 VBUS is switched ´by USB C PD controller on sheet "USB PD""
